File: blindscontrol.kicad_pcb (KiCad board)
At the start: 2 copper layers, 86.2 x 139.8 mm, 29 parts, among them SW1 SW_SPST, U1 Pico

Commit message: made some changes
Also trying to export it for fusion360 so I can make a case around it
Connections:
- U1 pad 13: unconnected-(U1-GND-Pad13) -> GND
Routing:
- added copper zone on B.Cu, net GND
- added copper zone on F.Cu, net GND
Changed lines of the file:
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@@
   (net 2 "unconnected-(U1-GND-Pad8)")
   (net 3 "unconnected-(U1-GPIO9-Pad12)")
-  (net 4 "unconnected-(U1-GND-Pad13)")
+  (net 4 "GND")
   (net 5 "unconnected-(U1-GND-Pad18)")
   (net 6 "unconnected-(U1-GPIO14-Pad19)")
@@
       (net 3 "unconnected-(U1-GPIO9-Pad12)") (pinfunction "GPIO9") (pintype "bidirectional"))
     (pad "13" thru_hole rect (at -8.89 6.35 90) (size 1.7 1.7) (drill 1.02) (layers "*.Cu" "*.Mask")
-      (net 4 "unconnected-(U1-GND-Pad13)") (pinfunction "GND") (pintype "power_in"))
+      (net 4 "GND") (pinfunction "GND") (pintype "power_in"))
     (pad "13" smd rect (at -8.89 6.35 90) (size 3.5 1.7) (drill (offset -0.9 0)) (layers "F.Cu" "F.Mask")
-      (net 4 "unconnected-(U1-GND-Pad13)") (pinfunction "GND") (pintype "power_in"))
+      (net 4 "GND") (pinfunction "GND") (pintype "power_in"))
     (pad "14" thru_hole oval (at -8.89 8.89 90) (size 1.7 1.7) (drill 1.02) (layers "*.Cu" "*.Mask")
       (net 27 "unconnected-(U1-GPIO10-Pad14)") (pinfunction "GPIO10") (pintype "bidirectional"))
@@
   (gr_circle (center 273.05 226.06) (end 273.05 227.584)
     (stroke (width 0.1) (type default)) (fill none) (layer "Edge.Cuts"))
-  (gr_text "Blinds Controller for HA V1 By Neptune" (at 270.129 225.171) (layer "B.SilkS")
+  (gr_text "Blinds Controller for HA V1 By Neptune" (at 224.663 225.171) (layer "B.SilkS")
     (effects (font (size 1 1) (thickness 0.15)) (justify left bottom mirror))
   )
@@
   (segment (start 207.546 152.355255) (end 207.546 138.331) (width 0.25) (layer "F.Cu") (net 57))
   (segment (start 225.171 122.047) (end 228.482 118.736) (width 0.25) (layer "F.Cu") (net 57))
+  (zone (net 4) (net_name "GND") (layers "F&B.Cu") (hatch edge 0.5)
+    (connect_pads (clearance 0.5))
+    (min_thickness 0.25) (filled_areas_thickness no)
+    (fill yes (thermal_gap 0.5) (thermal_bridge_width 0.5))
+    (polygon
+      (pts
+        (xy 184.15 122.555)
+        (xy 286.893 122.301)
+        (xy 283.972 235.585)
+        (xy 181.229 232.918)
+        (xy 184.277 122.428)
+      )
+    )
+  )
 )
