File: blindscontrol.kicad_sch (KiCad schematic)
At the start: 29 parts, among them SW1 SW_SPST, U1 Pico

Commit message: made some changes
Also trying to export it for fusion360 so I can make a case around it
Connections:
- net GND: now reaches U1.13 (GND)
Changed lines of the file:
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@@
+    )
+  )
+  (symbol (lib_id "power:GND") (at 30.48 77.47 270) (unit 1)
+    (in_bom yes) (on_board yes) (dnp no) (fields_autoplaced)
+    (property "Reference" "#PWR01" (at 24.13 77.47 0)
+      (effects (font (size 1.27 1.27)) hide)
+    )
+    (property "Value" "GND" (at 26.67 77.47 90)
+      (effects (font (size 1.27 1.27)) (justify right))
+    )
+    (property "Footprint" "" (at 30.48 77.47 0)
+      (effects (font (size 1.27 1.27)) hide)
+    )
+    (property "Datasheet" "" (at 30.48 77.47 0)
+      (effects (font (size 1.27 1.27)) hide)
+    )
+    (pin "1")
+    (instances
+      (project "blindscontrol"
+        (path "/2442bc7e-a5bc-44bc-b994-f17186191854"
+          (reference "#PWR01") (unit 1)
+        )
+      )
     )
   )
